File: pcb/puenteH/puenteH.sch (KiCad schematic (older format))
At the start: 25 parts, among them P1 CONN_2, Q1 DARL_P, Q2 DARL_N, Q3 DARL_P, Q4 DARL_N, U1 OPTO-TRANSISTOR4, U2 OPTO-TRANSISTOR4, U3 OPTO-TRANSISTOR4, U4 OPTO-TRANSISTOR4

Commit message: Complete table of true
Parts:
- R1, R11, R12, R2: value R -> 470
Other:
- note added: "0"
- note added: "1"
- note added: "Adelante"
- note added: "Atrás"
- note added: "Fijo"
- note added: "Freno motor"
- note added: "Nota: Con esta configuración de pines, \nobservar que no hay estados prohibidos, \no sea que nunca conducen a la vez un \ntransitor PNP con uno NPN que pongan \nen corto circutito fuente con tierra."
- note added: "X"
Changed lines of the file:
@@
-EESchema Schematic File Version 2  date mar 18 dic 2012 18:30:23 UYST
+EESchema Schematic File Version 2  date vie 21 dic 2012 21:28:10 UYST
 LIBS:power
 LIBS:device
@@
 Sheet 1 1
 Title "Puente H para motores CC"
-Date "18 dec 2012"
+Date "21 dec 2012"
 Rev "1.0"
 Comp ""
@@
 Comment4 ""
 $EndDescr
+Wire Wire Line
+	1900 4300 1100 4300
+Wire Notes Line
+	9120 470  9120 7200
+Wire Wire Line
+	6450 3100 6450 3200
+Wire Wire Line
+	5950 3100 5800 3100
+Wire Wire Line
+	6450 4300 6450 4450
+Wire Wire Line
+	5800 4800 5800 4450
+Wire Wire Line
+	3150 4300 3150 4450
+Wire Wire Line
+	4300 4800 4300 4650
+Wire Wire Line
+	3800 4450 3650 4450
+Wire Wire Line
+	1100 3500 1900 3500
+Wire Wire Line
+	3800 2750 3650 2750
+Wire Wire Line
+	3650 2750 3650 3100
+Wire Wire Line
+	5100 2750 4500 2750
+Wire Wire Line
+	7700 3500 8550 3500
+Wire Wire Line
+	6450 3500 6450 3650
+Wire Wire Line
+	3150 3500 3150 3650
+Wire Wire Line
+	7700 4000 7850 4000
+Wire Wire Line
+	1750 4000 1900 4000
+Wire Wire Line
+	1750 3200 1900 3200
+Wire Wire Line
+	5400 3300 5100 3300
+Wire Wire Line
+	5100 3300 5100 4250
+Wire Wire Line
+	4500 4250 4500 3300
+Wire Wire Line
+	4700 5400 4900 5400
+Connection ~ 4800 4800
+Wire Wire Line
+	4800 4900 4800 4800
+Wire Wire Line
+	4500 4800 5100 4800
+Wire Wire Line
+	4500 4800 4500 4650
+Wire Wire Line
+	5100 2750 5100 2900
+Wire Wire Line
+	5100 4650 5300 4650
+Wire Wire Line
+	4500 4250 4200 4250
+Wire Wire Line
+	4500 2900 4300 2900
+Wire Wire Line
+	5100 2900 5300 2900
+Wire Wire Line
+	4500 3300 4200 3300
+Wire Wire Line
+	5100 4250 5400 4250
+Wire Wire Line
+	4500 4650 4300 4650
+Wire Wire Line
+	5100 4650 5100 4800
+Wire Wire Line
+	4500 2900 4500 2750
+Wire Wire Line
+	4800 2600 4800 2750
+Connection ~ 4800 2750
+Wire Wire Line
+	4700 5600 4900 5600
+Wire Wire Line
+	4600 3750 4500 3750
+Connection ~ 4500 3750
+Wire Wire Line
+	5000 3750 5100 3750
+Connection ~ 5100 3750
+Wire Wire Line
+	7700 3200 7850 3200
+Wire Wire Line
+	3150 3900 3150 4000
+Wire Wire Line
+	6450 3900 6450 4000
+Wire Wire Line
+	8550 4000 8350 4000
+Wire Wire Line
+	1100 4000 1250 4000
+Wire Wire Line
+	8350 3200 8550 3200
+Wire Wire Line
+	3650 3100 3800 3100
+Wire Wire Line
+	1100 3200 1250 3200
+Wire Wire Line
+	3650 4450 3650 4800
+Wire Wire Line
+	3650 4800 3800 4800
+Wire Wire Line
+	4300 2900 4300 2750
+Wire Wire Line
+	5800 4450 5950 4450
+Wire Wire Line
+	5300 4650 5300 4800
+Wire Wire Line
+	5800 3100 5800 2750
+Wire Wire Line
+	5300 2900 5300 2750
+Wire Wire Line
+	3150 3100 3150 3200
+Wire Wire Line
+	7700 4300 8550 4300
+Text Notes 9250 2300 0    60   ~ 0
+Nota: Con esta configuración de pines, \nobservar que no hay estados prohibidos, \no sea que nunca conducen a la vez un \ntransitor PNP con uno NPN que pongan \nen corto circutito fuente con tierra.
+Text Notes 10500 1600 0    60   ~ 0
+Freno motor
+Text Notes 9400 1600 0    60   ~ 0
+1
+Text Notes 9750 1600 0    60   ~ 0
+1
+Text Notes 10100 1600 0    60   ~ 0
+0
+Text Notes 10500 1900 0    60   ~ 0
+Fijo
+Text Notes 10100 1900 0    60   ~ 0
+1
+Text Notes 9750 1900 0    60   ~ 0
+X
+Text Notes 9400 1900 0    60   ~ 0
+X
+Text Notes 10500 1750 0    60   ~ 0
+Fijo
+Text Notes 10100 1750 0    60   ~ 0
+X
+Text Notes 9750 1750 0    60   ~ 0
+0
+Text Notes 9400 1750 0    60   ~ 0
+0
+Text Notes 10500 1450 0    60   ~ 0
+Atrás
+Text Notes 10100 1450 0    60   ~ 0
+0
+Text Notes 9750 1450 0    60   ~ 0
+1
+Text Notes 9400 1450 0    60   ~ 0
+0
+Text Notes 10500 1300 0    60   ~ 0
+Adelante
+Text Notes 10100 1300 0    60   ~ 0
+0
+Text Notes 9750 1300 0    60   ~ 0
+0
+Text Notes 9400 1300 0    60   ~ 0
+1
 Text Notes 10430 1130 0    60   ~ 0
 Movimiento
@@
 Text Notes 9350 770  0    60   ~ 0
 Tabla de verdad
-Wire Notes Line
-	9120 470  9120 7200
-Wire Wire Line
-	6450 3100 6450 3200
-Wire Wire Line
-	5950 3100 5800 3100
-Wire Wire Line
-	6450 4300 6450 4450
-Wire Wire Line
-	5800 4800 5800 4450
-Wire Wire Line
-	3150 4300 3150 4450
-Wire Wire Line
-	4300 4800 4300 4650
-Wire Wire Line
-	3800 4450 3650 4450
-Wire Wire Line
-	1100 3500 1900 3500
-Wire Wire Line
-	3800 2750 3650 2750
-Wire Wire Line
-	3650 2750 3650 3100
-Wire Wire Line
-	5100 2750 4500 2750
-Wire Wire Line
-	7700 3500 8550 3500
-Wire Wire Line
-	8550 4300 7700 4300
-Wire Wire Line
-	1900 4300 1100 4300
-Wire Wire Line
-	6450 3500 6450 3650
-Wire Wire Line
-	3150 3500 3150 3650
-Wire Wire Line
-	7700 4000 7850 4000
-Wire Wire Line
-	1750 4000 1900 4000
-Wire Wire Line
-	1750 3200 1900 3200
-Wire Wire Line
-	5400 3300 5100 3300
-Wire Wire Line
-	5100 3300 5100 4250
-Wire Wire Line
-	4500 4250 4500 3300
-Wire Wire Line
-	4700 5400 4900 5400
-Connection ~ 4800 4800
-Wire Wire Line
-	4800 4900 4800 4800
-Wire Wire Line
-	4500 4800 5100 4800
-Wire Wire Line
-	4500 4800 4500 4650
-Wire Wire Line
-	5100 2750 5100 2900
-Wire Wire Line
-	5100 4650 5300 4650
-Wire Wire Line
-	4500 4250 4200 4250
-Wire Wire Line
-	4500 2900 4300 2900
-Wire Wire Line
-	5100 2900 5300 2900
-Wire Wire Line
-	4500 3300 4200 3300
-Wire Wire Line
-	5100 4250 5400 4250
-Wire Wire Line
-	4500 4650 4300 4650
-Wire Wire Line
-	5100 4650 5100 4800
-Wire Wire Line
-	4500 2900 4500 2750
-Wire Wire Line
-	4800 2600 4800 2750
-Connection ~ 4800 2750
-Wire Wire Line
-	4700 5600 4900 5600
-Wire Wire Line
-	4600 3750 4500 3750
-Connection ~ 4500 3750
-Wire Wire Line
-	5000 3750 5100 3750
-Connection ~ 5100 3750
-Wire Wire Line
-	7700 3200 7850 3200
-Wire Wire Line
-	3150 3900 3150 4000
-Wire Wire Line
-	6450 3900 6450 4000
-Wire Wire Line
-	8550 4000 8350 4000
-Wire Wire Line
-	1100 4000 1250 4000
-Wire Wire Line
-	8350 3200 8550 3200
-Wire Wire Line
-	3650 3100 3800 3100
-Wire Wire Line
-	1100 3200 1250 3200
-Wire Wire Line
-	3650 4450 3650 4800
-Wire Wire Line
-	3650 4800 3800 4800
-Wire Wire Line
-	4300 2900 4300 2750
-Wire Wire Line
-	5800 4450 5950 4450
-Wire Wire Line
-	5300 4650 5300 4800
-Wire Wire Line
-	5800 3100 5800 2750
-Wire Wire Line
-	5300 2900 5300 2750
-Wire Wire Line
-	3150 3100 3150 3200
 Text GLabel 1100 3500 0    60   Input ~ 0
 Inv
@@
 Dir
 $Comp
-L VCC #PWR6
+L VCC #PWR01
 U 1 1 50C7B069
 P 6450 3900
-F 0 "#PWR6" H 6450 4000 30  0001 C CNN
+F 0 "#PWR01" H 6450 4000 30  0001 C CNN
 F 1 "VCC" H 6450 4000 30  0000 C CNN
 	1    6450 3900
@@
 $EndComp
 $Comp
-L GND #PWR5
+L GND #PWR02
 U 1 1 50C7B05F
 P 6450 3650
-F 0 "#PWR5" H 6450 3650 30  0001 C CNN
+F 0 "#PWR02" H 6450 3650 30  0001 C CNN
 F 1 "GND" H 6450 3580 30  0001 C CNN
 	1    6450 3650
@@
 $EndComp
 $Comp
-L VCC #PWR2
+L VCC #PWR03
 U 1 1 50C7B04C
 P 3150 3900
-F 0 "#PWR2" H 3150 4000 30  0001 C CNN
+F 0 "#PWR03" H 3150 4000 30  0001 C CNN
 F 1 "VCC" H 3150 4000 30  0000 C CNN
 	1    3150 3900
@@
 $EndComp
 $Comp
-L GND #PWR1
+L GND #PWR04
 U 1 1 50C7B034
 P 3150 3650
-F 0 "#PWR1" H 3150 3650 30  0001 C CNN
+F 0 "#PWR04" H 3150 3650 30  0001 C CNN
 F 1 "GND" H 3150 3580 30  0001 C CNN
 	1    3150 3650
@@
 P 8100 4000
 F 0 "R12" V 8180 4000 50  0000 C CNN
-F 1 "R" V 8100 4000 50  0000 C CNN
+F 1 "470" V 8100 4000 50  0000 C CNN
 	1    8100 4000
 	0    -1   -1   0
@@
 P 8100 3200
 F 0 "R11" V 8180 3200 50  0000 C CNN
-F 1 "R" V 8100 3200 50  0000 C CNN
+F 1 "470" V 8100 3200 50  0000 C CNN
 	1    8100 3200
 	0    -1   -1   0
@@
 P 1500 3200
 F 0 "R1" V 1580 3200 50  0000 C CNN
-F 1 "R" V 1500 3200 50  0000 C CNN
+F 1 "470" V 1500 3200 50  0000 C CNN
 	1    1500 3200
 	0    -1   -1   0
@@
 P 1500 4000
 F 0 "R2" V 1580 4000 50  0000 C CNN
-F 1 "R" V 1500 4000 50  0000 C CNN
+F 1 "470" V 1500 4000 50  0000 C CNN
 	1    1500 4000
 	0    -1   -1   0
@@
 $EndComp
 $Comp
-L GND #PWR4
+L GND #PWR05
 U 1 1 50C79DFE
 P 4800 4900
-F 0 "#PWR4" H 4800 4900 30  0001 C CNN
+F 0 "#PWR05" H 4800 4900 30  0001 C CNN
 F 1 "GND" H 4800 4830 30  0001 C CNN
 	1    4800 4900
@@
 $EndComp
 $Comp
-L VCC #PWR3
+L VCC #PWR06
 U 1 1 50C79CA1
 P 4800 2600
-F 0 "#PWR3" H 4800 2700 30  0001 C CNN
+F 0 "#PWR06" H 4800 2700 30  0001 C CNN
 F 1 "VCC" H 4800 2700 30  0000 C CNN
 	1    4800 2600
